File: cpu_dma.kicad_sch (KiCad schematic)
At the start: 17 parts

Commit message: Updated to version 8
Changed to version 8; added 96-pin connectors; described ports at PPI_Settings
Parts:
- gave numbers to parts that had none: 17
