File: backplane.kicad_sch (KiCad schematic)
At the start: 2 parts, among them J1 ATX-20

Commit message: Added interrupts bus
Added interrupts bus
Connections:
- net VEE: no longer J1.18 (-5V/NC)
- new net VBB: J1.18 (-5V/NC)
Changed lines of the file:
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@@
 			)
 		)
-		(property "Value" "VEE"
+		(property "Value" "VBB"
 			(at 80.01 81.2799 90)
 			(effects
